Commit message: Added Camera Visuals

File: src/panda_gz_sim/urdf/panda_gz.urdf.xacro (robot description, xacro)
@@ -148,6 +148,6 @@
     <parent link="panda_hand"/>
     <child link="camera_link"/>
-    <!-- 8 cm below the hand centre, tilted 30° down to see the workspace -->
-    <origin xyz="0.0 0.0 -0.08" rpy="0 0.5236 0"/>
+    <!-- Move camera forward and lower to avoid clipping with the gripper fingers -->
+    <origin xyz="0.14 0.0 -0.12" rpy="0 -2.10 0"/>
   </joint>
   <!-- Optical frame (ROS image convention) -->
@@ -168,4 +168,5 @@
          /camera/depth/points           (sensor_msgs/PointCloud2)
   ============================================================ -->
+  <!-- Both sensors in a single gazebo block to avoid duplicate-reference issues -->
   <gazebo reference="camera_link">
     <sensor name="depth_camera" type="depth_camera">
@@ -174,5 +175,5 @@
       <visualize>true</visualize>
       <camera name="depth_camera">
-        <horizontal_fov>1.047</horizontal_fov>  <!-- 60 degrees -->
+        <horizontal_fov>1.047</horizontal_fov>
         <image>
           <width>640</width>
@@ -193,7 +194,4 @@
       <gz_frame_id>camera_depth_optical_frame</gz_frame_id>
     </sensor>
-  </gazebo>
-  <!-- Separate RGB camera (same body, for colour texture) -->
-  <gazebo reference="camera_link">
     <sensor name="rgb_camera" type="camera">
       <always_on>1</always_on>
@@ -205,5 +203,5 @@
           <width>640</width>
           <height>480</height>
-          <format>RGB_INT8</format>
+          <format>R8G8B8</format>
         </image>
         <clip>

Commit message: Added web camera viewer with Node, React, & ROS Bridge

File: src/panda_gz_sim/urdf/panda_gz.urdf.xacro (robot description, xacro)
@@ -148,6 +148,6 @@
     <parent link="panda_hand"/>
     <child link="camera_link"/>
-    <!-- Move camera forward and lower to avoid clipping with the gripper fingers -->
-    <origin xyz="0.14 0.0 -0.12" rpy="0 -2.10 0"/>
+    <!-- Camera positioned close below the hand, pointing straight down -->
+    <origin xyz="0.08 0.0 -0.10" rpy="0 -1.5708 0"/>
   </joint>
   <!-- Optical frame (ROS image convention) -->

Commit message: Minor Changes

File: src/panda_gz_sim/urdf/panda_gz.urdf.xacro (robot description, xacro)
@@ -149,5 +149,5 @@
     <child link="camera_link"/>
     <!-- Camera positioned close below the hand, pointing straight down -->
-    <origin xyz="0.08 0.0 -0.10" rpy="0 -1.5708 0"/>
+    <origin xyz="0.12 0.0 -0.10" rpy="0 -1.5708 0"/>
   </joint>
   <!-- Optical frame (ROS image convention) -->
@@ -192,5 +192,6 @@
       </camera>
       <topic>camera/depth</topic>
-      <gz_frame_id>camera_depth_optical_frame</gz_frame_id>
+      <camera_info_topic>camera/depth/camera_info</camera_info_topic>
+      <gz_frame_id>camera_link</gz_frame_id>
     </sensor>
     <sensor name="rgb_camera" type="camera">
@@ -211,5 +212,6 @@
       </camera>
       <topic>camera/color</topic>
-      <gz_frame_id>camera_depth_optical_frame</gz_frame_id>
+      <camera_info_topic>camera/color/camera_info</camera_info_topic>
+      <gz_frame_id>camera_link</gz_frame_id>
     </sensor>
   </gazebo>
